File: kicad/in-12-tester.sch (KiCad schematic (older format))
At the start: 68 parts, among them J1 Jack-DC, Q1 MMBTA92, Q10 MMBTA42, Q11 MMBTA42, Q12 MMBTA42, Q13 MMBTA42, Q14 MMBTA42, Q15 MMBTA42, Q16 MMBTA42, Q17 IRF740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

Commit message: Added tester schematic.
Parts:
- L1, L2: value ins-1 -> INS-1; footprint Parts:ins-1 -> PartsStash:INS-1; symbol parts_library:ins-1 -> Russian_Lamps:ins-1
- MK1, MK2, MK3, MK4: symbol Mechanical:Mounting_Hole -> Mechanical:MountingHole
- Q1, Q4: symbol parts_library:mmbta92 -> Parts_Stash:MMBTA92
- Q10, Q11, Q12, Q13, Q14, Q15, Q16, Q2, Q3, Q5, Q6, Q7, Q8, Q9: symbol parts_library:MMBTA42 -> Parts_Stash:MMBTA42
- T1: symbol parts_library:IN-12 -> Russian_Lamps:IN-12
- U1: symbol parts_library:max1771 -> Parts_Stash:MAX1771
- U3, U4, U5, U6, U7: symbol parts_library:THERMAL_VIA -> Parts_Stash:THERMAL_VIA
Connections:
- wire segments 200 -> 197
Changed lines of the file:
@@
 EESchema Schematic File Version 4
-LIBS:in-12-tester-cache
 EELAYER 26 0
 EELAYER END
@@
 $EndDescr
 $Comp
-L parts_library:IN-12 T1
+L Russian_Lamps:IN-12 T1
 U 1 1 5B499E3D
 P 2350 3500
@@
 $EndComp
 $Comp
-L parts_library:mmbta92 Q1
+L Parts_Stash:MMBTA92 Q1
 U 1 1 5B49A110
 P 2250 1650
@@
 $EndComp
 $Comp
-L parts_library:MMBTA42 Q2
+L Parts_Stash:MMBTA42 Q2
 U 1 1 5B49A7EF
 P 4500 6700
@@
 $EndComp
 $Comp
-L parts_library:ins-1 L1
+L Russian_Lamps:ins-1 L1
 U 1 1 5B49D974
 P 3550 1850
 F 0 "L1" V 3504 1974 50  0000 L CNN
-F 1 "ins-1" V 3595 1974 50  0000 L CNN
-F 2 "Parts:ins-1" V 3550 1850 50  0001 C CNN
+F 1 "INS-1" V 3595 1974 50  0000 L CNN
+F 2 "PartsStash:INS-1" V 3550 1850 50  0001 C CNN
 F 3 "" V 3550 1850 50  0001 C CNN
 	1    3550 1850
@@
 $EndComp
 $Comp
-L parts_library:MMBTA42 Q6
+L Parts_Stash:MMBTA42 Q6
 U 1 1 5B49DBDA
 P 2800 5100
@@
 Connection ~ 2350 1050
 $Comp
-L parts_library:mmbta92 Q4
+L Parts_Stash:MMBTA92 Q4
 U 1 1 5B4A1078
 P 4700 1500
@@
 $EndComp
 $Comp
-L parts_library:ins-1 L2
+L Russian_Lamps:ins-1 L2
 U 1 1 5B4A125B
 P 4600 2400
 F 0 "L2" V 4554 2524 50  0000 L CNN
-F 1 "ins-1" V 4645 2524 50  0000 L CNN
-F 2 "Parts:ins-1" V 4600 2400 50  0001 C CNN
+F 1 "INS-1" V 4645 2524 50  0000 L CNN
+F 2 "PartsStash:INS-1" V 4600 2400 50  0001 C CNN
 F 3 "" V 4600 2400 50  0001 C CNN
 	1    4600 2400
@@
 $EndComp
 $Comp
-L parts_library:MMBTA42 Q5
+L Parts_Stash:MMBTA42 Q5
 U 1 1 5B4A23C0
 P 1900 6750
@@
 	2900 4700 2900 4900
 $Comp
-L parts_library:MMBTA42 Q8
+L Parts_Stash:MMBTA42 Q8
 U 1 1 5B4B391D
 P 3650 5100
@@
 	3750 4700 3750 4900
 $Comp
-L parts_library:MMBTA42 Q7
+L Parts_Stash:MMBTA42 Q7
 U 1 1 5B4B51C2
 P 1000 5100
@@
 	1100 4850 1100 4900
 $Comp
-L parts_library:MMBTA42 Q9
+L Parts_Stash:MMBTA42 Q9
 U 1 1 5B4B6FA3
 P 4500 5100
@@
 	4600 4700 4600 4900
 $Comp
-L parts_library:MMBTA42 Q10
+L Parts_Stash:MMBTA42 Q10
 U 1 1 5B4B8120
 P 5350 5100
@@
 	5450 4700 5450 4900
 $Comp
-L parts_library:MMBTA42 Q11
+L Parts_Stash:MMBTA42 Q11
 U 1 1 5B4B9668
 P 2800 6750
@@
 	2900 6350 2900 6550
 $Comp
-L parts_library:MMBTA42 Q12
+L Parts_Stash:MMBTA42 Q12
 U 1 1 5B4BAEE4
 P 3650 6750
@@
 	3750 6350 3750 6550
 $Comp
-L parts_library:MMBTA42 Q13
+L Parts_Stash:MMBTA42 Q13
 U 1 1 5B4BCB82
 P 5250 2400
@@
 	5550 2400 5550 2450
 $Comp
-L parts_library:MMBTA42 Q14
+L Parts_Stash:MMBTA42 Q14
 U 1 1 5B4BEC46
 P 3450 2400
@@
 	3150 2400 3150 2450
 $Comp
-L parts_library:MMBTA42 Q15
+L Parts_Stash:MMBTA42 Q15
 U 1 1 5B4C10E0
 P 1900 5100
@@
 	2000 4700 2000 4900
 $Comp
-L parts_library:MMBTA42 Q16
+L Parts_Stash:MMBTA42 Q16
 U 1 1 5B4CAFAB
 P 1750 2400
@@
 $EndComp
 $Comp
-L parts_library:MMBTA42 Q3
+L Parts_Stash:MMBTA42 Q3
 U 1 1 5B4D7431
 P 1000 6750
@@
 	6450 850  6450 750
 $Comp
-L parts_library:max1771 U1
+L Parts_Stash:MAX1771 U1
 U 1 1 5B71C581
 P 7900 2600
@@
 Connection ~ 10600 1500
 $Comp
-L Mechanical:Mounting_Hole MK1
+L Mechanical:MountingHole MK1
 U 1 1 5B9313A3
 P 8900 4450
@@
 $EndComp
 $Comp
-L Mechanical:Mounting_Hole MK3
+L Mechanical:MountingHole MK3
 U 1 1 5B9314D3
 P 9300 4450
@@
 $EndComp
 $Comp
-L Mechanical:Mounting_Hole MK4
+L Mechanical:MountingHole MK4
 U 1 1 5B931565
 P 9300 4750
@@
 $EndComp
 $Comp
-L Mechanical:Mounting_Hole MK2
+L Mechanical:MountingHole MK2
 U 1 1 5B9315FD
 P 8900 4750
@@
 	3550 2100 3550 2200
 $Comp
-L parts_library:THERMAL_VIA U3
+L Parts_Stash:THERMAL_VIA U3
 U 1 1 5BA2A652
 P 8900 5100
@@
 $EndComp
 $Comp
-L parts_library:THERMAL_VIA U4
+L Parts_Stash:THERMAL_VIA U4
 U 1 1 5BA2A731
 P 9100 5100
@@
 $EndComp
 $Comp
-L parts_library:THERMAL_VIA U5
+L Parts_Stash:THERMAL_VIA U5
 U 1 1 5BA34D07
 P 9300 5100
@@
 $EndComp
 $Comp
-L parts_library:THERMAL_VIA U6
+L Parts_Stash:THERMAL_VIA U6
 U 1 1 5BA34D90
 P 9500 5100
@@
 $EndComp
 $Comp
-L parts_library:THERMAL_VIA U7
+L Parts_Stash:THERMAL_VIA U7
 U 1 1 5BA34E19
 P 9700 5100
@@
 	1    0    0    -1
 $EndComp
-Wire Wire Line
-	9700 5200 9500 5200
-Wire Wire Line
-	9500 5200 9300 5200
-Connection ~ 9500 5200
-Wire Wire Line
-	9300 5200 9100 5200
-Connection ~ 9300 5200
-Wire Wire Line
-	9100 5200 8900 5200
-Connection ~ 9100 5200
 $Comp
 L power:GND #PWR0102
@@
 Wire Wire Line
 	8900 5300 8900 5200
-Connection ~ 8900 5200
+Wire Wire Line
+	8900 5200 9700 5200
 $EndSCHEMATC
